File: src/LEDx11.kicad_sch (KiCad schematic)
At the start: 22 parts

Commit message: Add: Vendor no. and footprints
Parts:
- C801, C802, C803, C804, C805, C806, C807, C808, C809, C810, C811: footprint (none) -> Capacitor_SMD:C_0805_2012Metric_Pad1.18x1.45mm_HandSolder; Manufacturer (none) -> -; Manufacturer Part no. (none) -> -; Vendor 1 (none) -> Digikey; Vendor 1 Part no. (none) -> 1276-2444-1-ND; Vendor 2 (none) -> LCSC

Commit message: Mod: Changed parts to match with both vendors
Parts:
- C801, C802, C803, C804, C805, C806, C807, C808, C809, C810, C811: Manufacturer - -> Samsung Electro-Mechanics; Manufacturer Part no. - -> CL21B104KBCNFNC; Vendor 2 Part no. (none) -> C318718
- D801, D802, D803, D804, D805, D806, D807, D808, D809, D810, D811: Manufacturer SparkFun Electronics -> -; Manufacturer Part no. COM-16347 -> WS2812B; Vendor 2 Part no. C114586 -> C22461793
