File: src/LEDx4.kicad_sch (KiCad schematic)
At the start: 8 parts

Commit message: Add: Vendor no. and footprints
Parts:
- C701, C702, C703, C704: footprint (none) -> Capacitor_SMD:C_0805_2012Metric_Pad1.18x1.45mm_HandSolder; Manufacturer (none) -> -; Manufacturer Part no. (none) -> -; Vendor 1 (none) -> Digikey; Vendor 1 Part no. (none) -> 1276-2444-1-ND; Vendor 2 (none) -> LCSC
Changed lines of the file:
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@@
 			)
 		)
-		(property "Footprint" ""
+		(property "Footprint" "Capacitor_SMD:C_0805_2012Metric_Pad1.18x1.45mm_HandSolder"
 			(at 127.9652 181.61 0)
 			(effects
@@
 		)
 		(property "Sim.Type" ""
+			(at 127 177.8 0)
+			(effects
+				(font
+					(size 1.27 1.27)
+				)
+				(hide yes)
+			)
+		)
+		(property "Manufacturer" "-"
+			(at 127 177.8 0)
+			(effects
+				(font
+					(size 1.27 1.27)
+				)
+				(hide yes)
+			)
+		)
+		(property "Manufacturer Part no." "-"
+			(at 127 177.8 0)
+			(effects
+				(font
+					(size 1.27 1.27)
+				)
+				(hide yes)
+			)
+		)
+		(property "Vendor 1" "Digikey"
+			(at 127 177.8 0)
+			(effects
+				(font
+					(size 1.27 1.27)
+				)
+				(hide yes)
+			)
+		)
+		(property "Vendor 1 Part no." "1276-2444-1-ND "
+			(at 127 177.8 0)
+			(effects
+				(font
+					(size 1.27 1.27)
+				)
+				(hide yes)
+			)
+		)
+		(property "Vendor 2" "LCSC"
 			(at 127 177.8 0)
 			(effects
@@
 			)
 		)
-		(property "Footprint" ""
+		(property "Footprint" "Capacitor_SMD:C_0805_2012Metric_Pad1.18x1.45mm_HandSolder"
 			(at 140.6652 181.61 0)
 			(effects
@@
 		)
 		(property "Sim.Type" ""
+			(at 139.7 177.8 0)
+			(effects
+				(font
+					(size 1.27 1.27)
+				)
+				(hide yes)
+			)
+		)
+		(property "Manufacturer" "-"
+			(at 139.7 177.8 0)
+			(effects
+				(font
+					(size 1.27 1.27)
+				)
+				(hide yes)
+			)
+		)
+		(property "Manufacturer Part no." "-"
+			(at 139.7 177.8 0)
+			(effects
+				(font
+					(size 1.27 1.27)
+				)
+				(hide yes)
+			)
+		)
+		(property "Vendor 1" "Digikey"
+			(at 139.7 177.8 0)
+			(effects
+				(font
+					(size 1.27 1.27)
+				)
+				(hide yes)
+			)
+		)
+		(property "Vendor 1 Part no." "1276-2444-1-ND "
+			(at 139.7 177.8 0)
+			(effects
+				(font
+					(size 1.27 1.27)
+				)
+				(hide yes)
+			)
+		)
+		(property "Vendor 2" "LCSC"
 			(at 139.7 177.8 0)
 			(effects
@@
 			)
 		)
-		(property "Footprint" ""
+		(property "Footprint" "Capacitor_SMD:C_0805_2012Metric_Pad1.18x1.45mm_HandSolder"
 			(at 153.3652 181.61 0)
 			(effects
@@
 		)
 		(property "Sim.Type" ""
+			(at 152.4 177.8 0)
+			(effects
+				(font
+					(size 1.27 1.27)
+				)
+				(hide yes)
+			)
+		)
+		(property "Manufacturer" "-"
+			(at 152.4 177.8 0)
+			(effects
+				(font
+					(size 1.27 1.27)
+				)
+				(hide yes)
+			)
+		)
+		(property "Manufacturer Part no." "-"
+			(at 152.4 177.8 0)
+			(effects
+				(font
+					(size 1.27 1.27)
+				)
+				(hide yes)
+			)
+		)
+		(property "Vendor 1" "Digikey"
+			(at 152.4 177.8 0)
+			(effects
+				(font
+					(size 1.27 1.27)
+				)
+				(hide yes)
+			)
+		)
+		(property "Vendor 1 Part no." "1276-2444-1-ND "
+			(at 152.4 177.8 0)
+			(effects
+				(font
+					(size 1.27 1.27)
+				)
+				(hide yes)
+			)
+		)
+		(property "Vendor 2" "LCSC"
 			(at 152.4 177.8 0)
 			(effects
@@
 			)
 		)
-		(property "Footprint" ""
+		(property "Footprint" "Capacitor_SMD:C_0805_2012Metric_Pad1.18x1.45mm_HandSolder"
 			(at 166.0652 181.61 0)
 			(effects
@@
 			(at 165.1 177.8 0)
 			(effects
+				(font
+					(size 1.27 1.27)
+				)
+				(hide yes)
+			)
+		)
+		(property "Manufacturer" "-"
+			(at 165.1 177.8 0)
+			(effects
+				(font
+					(size 1.27 1.27)
+				)
+				(hide yes)
+			)
+		)
+		(property "Manufacturer Part no." "-"
+			(at 165.1 177.8 0)
+			(effects
+				(font
+					(size 1.27 1.27)
+				)
+				(hide yes)
+			)
+		)
+		(property "Vendor 1" "Digikey"
+			(at 165.1 177.8 0)
+			(effects
+				(font
+					(size 1.27 1.27)
+				)
+				(hide yes)
+			)
+		)
+		(property "Vendor 1 Part no." "1276-2444-1-ND "
+			(at 165.1 177.8 0)
+			(effects
+				(font
+					(size 1.27 1.27)
+				)
+				(hide yes)
+			)
+		)
+		(property "Vendor 2" "LCSC"
+			(at 165.1 177.8 0)
+			(effects

Commit message: Mod: Changed parts to match with both vendors
Parts:
- C701, C702, C703, C704: Manufacturer - -> Samsung Electro-Mechanics; Manufacturer Part no. - -> CL21B104KBCNFNC; Vendor 2 Part no. (none) -> C318718
- D701, D702, D703, D704: Manufacturer SparkFun Electronics -> -; Manufacturer Part no. COM-16347 -> WS2812B; Vendor 2 Part no. C114586 -> C22461793
Changed lines of the file:
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@@
 	(title_block
 		(title "Wordclock - LED Row with 4 pcs.")
-		(date "2024-10-27")
+		(date "2024-10-29")
 		(rev "A")
 		(company "ElektroNik Zoller")
@@
 			)
 		)
-		(property "Manufacturer" "-"
+		(property "Manufacturer" "Samsung Electro-Mechanics"
 			(at 127 177.8 0)
 			(effects
@@
 			)
 		)
-		(property "Manufacturer Part no." "-"
+		(property "Manufacturer Part no." "CL21B104KBCNFNC"
 			(at 127 177.8 0)
 			(effects
@@
 		)
 		(property "Vendor 2" "LCSC"
+			(at 127 177.8 0)
+			(effects
+				(font
+					(size 1.27 1.27)
+				)
+				(hide yes)
+			)
+		)
+		(property "Vendor 2 Part no." "C318718"
 			(at 127 177.8 0)
 			(effects
@@
 			)
 		)
-		(property "Manufacturer" "-"
+		(property "Manufacturer" "Samsung Electro-Mechanics"
 			(at 139.7 177.8 0)
 			(effects
@@
 			)
 		)
-		(property "Manufacturer Part no." "-"
+		(property "Manufacturer Part no." "CL21B104KBCNFNC"
 			(at 139.7 177.8 0)
 			(effects
@@
 		)
 		(property "Vendor 2" "LCSC"
+			(at 139.7 177.8 0)
+			(effects
+				(font
+					(size 1.27 1.27)
+				)
+				(hide yes)
+			)
+		)
+		(property "Vendor 2 Part no." "C318718"
 			(at 139.7 177.8 0)
 			(effects
@@
 			)
 		)
-		(property "Manufacturer" "SparkFun Electronics"
+		(property "Manufacturer" "-"
 			(at 127 50.8 0)
 			(effects
@@
 			)
 		)
-		(property "Manufacturer Part no." "COM-16347"
+		(property "Manufacturer Part no." "WS2812B"
 			(at 127 50.8 0)
 			(effects
@@
 			)
 		)
-		(property "Vendor 2 Part no." "C114586"
+		(property "Vendor 2 Part no." "C22461793"
 			(at 127 50.8 0)
 			(effects
@@
 			)
 		)
-		(property "Manufacturer" "SparkFun Electronics"
+		(property "Manufacturer" "-"
 			(at 177.8 50.8 0)
 			(effects
@@
 			)
 		)
-		(property "Manufacturer Part no." "COM-16347"
+		(property "Manufacturer Part no." "WS2812B"
 			(at 177.8 50.8 0)
 			(effects
@@
 			)
 		)
-		(property "Vendor 2 Part no." "C114586"
+		(property "Vendor 2 Part no." "C22461793"
 			(at 177.8 50.8 0)
 			(effects
@@
 			)
 		)
-		(property "Manufacturer" "SparkFun Electronics"
+		(property "Manufacturer" "-"
 			(at 101.6 50.8 0)
 			(effects
@@
 			)
 		)
-		(property "Manufacturer Part no." "COM-16347"
+		(property "Manufacturer Part no." "WS2812B"
 			(at 101.6 50.8 0)
 			(effects
@@
 			)
 		)
-		(property "Vendor 2 Part no." "C114586"
+		(property "Vendor 2 Part no." "C22461793"
 			(at 101.6 50.8 0)
 			(effects
@@
 			)
 		)
-		(property "Manufacturer" "-"
+		(property "Manufacturer" "Samsung Electro-Mechanics"
 			(at 152.4 177.8 0)
 			(effects
@@
 			)
 		)
-		(property "Manufacturer Part no." "-"
+		(property "Manufacturer Part no." "CL21B104KBCNFNC"
 			(at 152.4 177.8 0)
 			(effects
@@
 		)
 		(property "Vendor 2" "LCSC"
+			(at 152.4 177.8 0)
+			(effects
+				(font
+					(size 1.27 1.27)
+				)
+				(hide yes)
+			)
+		)
+		(property "Vendor 2 Part no." "C318718"
 			(at 152.4 177.8 0)
 			(effects
@@
 			)
 		)
-		(property "Manufacturer" "-"
+		(property "Manufacturer" "Samsung Electro-Mechanics"
 			(at 165.1 177.8 0)
 			(effects
@@
 			)
 		)
-		(property "Manufacturer Part no." "-"
+		(property "Manufacturer Part no." "CL21B104KBCNFNC"
 			(at 165.1 177.8 0)
 			(effects
@@
 		)
 		(property "Vendor 2" "LCSC"
+			(at 165.1 177.8 0)
+			(effects
+				(font
+					(size 1.27 1.27)
+				)
+				(hide yes)
+			)
+		)
+		(property "Vendor 2 Part no." "C318718"
 			(at 165.1 177.8 0)
 			(effects
@@
 			)
 		)
-		(property "Manufacturer" "SparkFun Electronics"
+		(property "Manufacturer" "-"
 			(at 152.4 50.8 0)
 			(effects
@@
 			)
 		)
-		(property "Manufacturer Part no." "COM-16347"
+		(property "Manufacturer Part no." "WS2812B"
 			(at 152.4 50.8 0)
 			(effects
@@
 			)
 		)
-		(property "Vendor 2 Part no." "C114586"
+		(property "Vendor 2 Part no." "C22461793"
 			(at 152.4 50.8 0)
 			(effects
