File: src/LEDx4.kicad_sch (KiCad schematic)
At the start: 8 parts

Commit message: Add: JLCPCB Database and selected components for the assembly
Parts:
- C701, C702, C703, C704: Comment (none) -> Best fit from the JLCPCB "Basic" compontens; Manufacturer Part no. CL21B104KBCNFNC -> CL21B104KCFNNNE; Vendor 1 Part no. 1276-2444-1-ND -> 1276-6840-1-ND; Vendor 2 Part no. C318718 -> C28233
- D701, D702, D703, D704: LCSC (none) -> C22461793
Changed lines of the file:
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@@
 	(title_block
 		(title "Wordclock - LED Row with 4 pcs.")
-		(date "2024-11-01")
+		(date "2024-11-17")
 		(rev "A")
 		(company "ElektroNik Zoller")
@@
 			)
 		)
-		(property "Manufacturer Part no." "CL21B104KBCNFNC"
+		(property "Manufacturer Part no." "CL21B104KCFNNNE"
 			(at 127 177.8 0)
 			(effects
@@
 			)
 		)
-		(property "Vendor 1 Part no." "1276-2444-1-ND "
+		(property "Vendor 1 Part no." "1276-6840-1-ND"
 			(at 127 177.8 0)
 			(effects
@@
 			)
 		)
-		(property "Vendor 2 Part no." "C318718"
+		(property "Vendor 2 Part no." "C28233"
+			(at 127 177.8 0)
+			(effects
+				(font
+					(size 1.27 1.27)
+				)
+				(hide yes)
+			)
+		)
+		(property "Comment" "Best fit from the JLCPCB \"Basic\" compontens"
 			(at 127 177.8 0)
 			(effects
@@
 			)
 		)
-		(property "Manufacturer Part no." "CL21B104KBCNFNC"
+		(property "Manufacturer Part no." "CL21B104KCFNNNE"
 			(at 139.7 177.8 0)
 			(effects
@@
 			)
 		)
-		(property "Vendor 1 Part no." "1276-2444-1-ND "
+		(property "Vendor 1 Part no." "1276-6840-1-ND"
 			(at 139.7 177.8 0)
 			(effects
@@
 			)
 		)
-		(property "Vendor 2 Part no." "C318718"
+		(property "Vendor 2 Part no." "C28233"
+			(at 139.7 177.8 0)
+			(effects
+				(font
+					(size 1.27 1.27)
+				)
+				(hide yes)
+			)
+		)
+		(property "Comment" "Best fit from the JLCPCB \"Basic\" compontens"
 			(at 139.7 177.8 0)
 			(effects
@@
 			)
 		)
+		(property "LCSC" "C22461793"
+			(at 0 101.6 0)
+			(effects
+				(font
+					(size 1.27 1.27)
+				)
+				(hide yes)
+			)
+		)
 		(pin "2"
 		)
@@
 			)
 		)
+		(property "LCSC" "C22461793"
+			(at 0 101.6 0)
+			(effects
+				(font
+					(size 1.27 1.27)
+				)
+				(hide yes)
+			)
+		)
 		(pin "2"
 		)
@@
 			)
 		)
+		(property "LCSC" "C22461793"
+			(at 0 101.6 0)
+			(effects
+				(font
+					(size 1.27 1.27)
+				)
+				(hide yes)
+			)
+		)
 		(pin "2"
 		)
@@
 			)
 		)
-		(property "Manufacturer Part no." "CL21B104KBCNFNC"
+		(property "Manufacturer Part no." "CL21B104KCFNNNE"
 			(at 152.4 177.8 0)
 			(effects
@@
 			)
 		)
-		(property "Vendor 1 Part no." "1276-2444-1-ND "
+		(property "Vendor 1 Part no." "1276-6840-1-ND"
 			(at 152.4 177.8 0)
 			(effects
@@
 			)
 		)
-		(property "Vendor 2 Part no." "C318718"
+		(property "Vendor 2 Part no." "C28233"
+			(at 152.4 177.8 0)
+			(effects
+				(font
+					(size 1.27 1.27)
+				)
+				(hide yes)
+			)
+		)
+		(property "Comment" "Best fit from the JLCPCB \"Basic\" compontens"
 			(at 152.4 177.8 0)
 			(effects
@@
 			)
 		)
-		(property "Manufacturer Part no." "CL21B104KBCNFNC"
+		(property "Manufacturer Part no." "CL21B104KCFNNNE"
 			(at 165.1 177.8 0)
 			(effects
@@
 			)
 		)
-		(property "Vendor 1 Part no." "1276-2444-1-ND "
+		(property "Vendor 1 Part no." "1276-6840-1-ND"
 			(at 165.1 177.8 0)
 			(effects
@@
 			)
 		)
-		(property "Vendor 2 Part no." "C318718"
+		(property "Vendor 2 Part no." "C28233"
+			(at 165.1 177.8 0)
+			(effects
+				(font
+					(size 1.27 1.27)
+				)
+				(hide yes)
+			)
+		)
+		(property "Comment" "Best fit from the JLCPCB \"Basic\" compontens"
 			(at 165.1 177.8 0)
 			(effects
@@
 			(effects
 				(font
+					(size 1.27 1.27)
+				)
+				(hide yes)
+			)
+		)
+		(property "LCSC" "C22461793"
+			(at 0 101.6 0)
+			(effects
+				(font

Commit message: Mod: Updated date and fixed some typo
Parts:
- C701, C702, C703, C704: Comment Best fit from the JLCPCB "Basic" compontens -> Best fit from the JLCPCB "Basic" components
Changed lines of the file:
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@@
 	(title_block
 		(title "Wordclock - LED Row with 4 pcs.")
-		(date "2024-11-17")
+		(date "2024-11-25")
 		(rev "A")
 		(company "ElektroNik Zoller")
@@
 			)
 		)
-		(property "Comment" "Best fit from the JLCPCB \"Basic\" compontens"
+		(property "Comment" "Best fit from the JLCPCB \"Basic\" components"
 			(at 127 177.8 0)
 			(effects
@@
 			)
 		)
-		(property "Comment" "Best fit from the JLCPCB \"Basic\" compontens"
+		(property "Comment" "Best fit from the JLCPCB \"Basic\" components"
 			(at 139.7 177.8 0)
 			(effects
@@
 			)
 		)
-		(property "Comment" "Best fit from the JLCPCB \"Basic\" compontens"
+		(property "Comment" "Best fit from the JLCPCB \"Basic\" components"
 			(at 152.4 177.8 0)
 			(effects
@@
 			)
 		)
-		(property "Comment" "Best fit from the JLCPCB \"Basic\" compontens"
+		(property "Comment" "Best fit from the JLCPCB \"Basic\" components"
 			(at 165.1 177.8 0)
 			(effects
