File: src/USB.kicad_sch (KiCad schematic)
At the start: 29 parts, among them J301 USB_C_Receptacle_USB2.0_16P, Q301 NPN, Q302 NPN, U301 CP2102N-Axx-xQFN24

Commit message: Mod: Checked a few things and added the power limitation text to the LEDs page
Parts:
- renumbered C308 to C303, C303 to C304, C304 to C305, C305 to C306, C306 to C307, C307 to C308, R314 to R304, R313 to R305, R304 to R306, R305 to R307, R311 to R308, R312 to R309, R306 to R310, R307 to R311, R308 to R312, R309 to R313, R310 to R314
Other:
- moved on the sheet: R304, R305

Commit message: Mod: Changed the page number of the MCU and USB page
Parts:
- renumbered C301 to C210, C302 to C211, C303 to C212, C304 to C213, C305 to C214, C306 to C215, C307 to C216, C308 to C217, D301 to D203, D302 to D204, D303 to D205, J301 to J201, Q301 to Q201, Q302 to Q202, R301 to R205, R302 to R206, R303 to R207, R304 to R208, R305 to R209, R306 to R210, R307 to R211, R308 to R212, R309 to R213, R310 to R214, R311 to R215, R312 to R216, R313 to R217, R314 to R218, U301 to U203

Commit message: Fix: Some errors from the ERC
Parts:
- removed Q201, Q202: NPN, symbol Simulation_SPICE:NPN
- added Q201, Q202: NPN, Package_TO_SOT_SMD:SOT-23_Handsoldering, symbol Device:Q_NPN_BEC
- renumbered C210 to C201, C211 to C202, C212 to C203, C213 to C204, C214 to C205, C215 to C206, C216 to C207, C217 to C208, D203 to D201, D204 to D202, D205 to D203, R205 to R201, R206 to R202, R207 to R203, R208 to R204, R209 to R205, R210 to R206, R211 to R207, R212 to R208, R213 to R209, R214 to R210, R215 to R211, R216 to R212, R217 to R213, R218 to R214, U203 to U201
Connections:
- net BOOT: now also Q201.3 (C)
- net ~{RST}: now also Q202.3 (C)
- net at R211.1: now also Q201.1 (B)
- net at R211.2, U201.19 (~{RTS}): now also Q202.2 (E)
- net at R212.2, U201.23 (~{DTR}): now also Q201.2 (E)
- net at R212.1: now also Q202.1 (B)

Commit message: Add: Vendor no. and footprints
Parts:
- C201: value 10nF -> 0.1µF; footprint (none) -> Capacitor_SMD:C_0805_2012Metric_Pad1.18x1.45mm_HandSolder; Manufacturer (none) -> -; Manufacturer Part no. (none) -> -; Vendor 1 (none) -> Digikey; Vendor 1 Part no. (none) -> 1276-2444-1-ND; Vendor 2 (none) -> LCSC
- C202, C204, C205: footprint (none) -> Capacitor_SMD:C_0805_2012Metric_Pad1.18x1.45mm_HandSolder; Manufacturer (none) -> -; Manufacturer Part no. (none) -> -; Vendor 1 (none) -> Digikey; Vendor 1 Part no. (none) -> 1276-1096-1-ND; Vendor 2 (none) -> LCSC
- C203: footprint (none) -> Capacitor_SMD:C_0805_2012Metric_Pad1.18x1.45mm_HandSolder; Manufacturer (none) -> -; Manufacturer Part no. (none) -> -; Vendor 1 (none) -> Digikey; Vendor 1 Part no. (none) -> 1276-1275-2-ND; Vendor 2 (none) -> LCSC
- C206, C207, C208: footprint (none) -> Capacitor_SMD:C_0805_2012Metric_Pad1.18x1.45mm_HandSolder; Manufacturer (none) -> -; Manufacturer Part no. (none) -> -; Vendor 1 (none) -> Digikey; Vendor 1 Part no. (none) -> 1276-2444-1-ND; Vendor 2 (none) -> LCSC
- D201: Manufacturer (none) -> -; Manufacturer Part no. (none) -> SP0503BAHTG; Vendor 1 (none) -> Digikey; Vendor 1 Part no. (none) -> F2715CT-ND; Vendor 2 (none) -> LCSC; Vendor 2 Part no. (none) -> C7074
- D202, D203: footprint (none) -> LED_SMD:LED_0805_2012Metric_Pad1.15x1.40mm_HandSolder; Manufacturer (none) -> -; Manufacturer Part no. (none) -> -; Vendor 1 (none) -> Digikey; Vendor 1 Part no. (none) -> 160-1423-1-ND; Vendor 2 (none) -> LCSC
- Q201, Q202: value NPN -> NPN BJT
- R201, R204, R205, R208, R209: footprint (none) -> Resistor_SMD:R_0805_2012Metric_Pad1.20x1.40mm_HandSolder; Manufacturer (none) -> -; Manufacturer Part no. (none) -> -; Vendor 1 (none) -> Digikey; Vendor 1 Part no. (none) -> 311-0.0ARCT-ND; Vendor 2 (none) -> LCSC
- R202, R203: footprint (none) -> Resistor_SMD:R_0805_2012Metric_Pad1.20x1.40mm_HandSolder; Manufacturer (none) -> -; Manufacturer Part no. (none) -> -; Vendor 1 (none) -> Digikey; Vendor 1 Part no. (none) -> 311-5.10KCRCT-ND; Vendor 2 (none) -> LCSC
- R206: footprint (none) -> Resistor_SMD:R_0805_2012Metric_Pad1.20x1.40mm_HandSolder; Manufacturer (none) -> -; Manufacturer Part no. (none) -> -; Vendor 1 (none) -> Digikey; Vendor 1 Part no. (none) -> 311-22.1KCRCT-ND; Vendor 2 (none) -> LCSC
- R207: footprint (none) -> Resistor_SMD:R_0805_2012Metric_Pad1.20x1.40mm_HandSolder; Manufacturer (none) -> -; Manufacturer Part no. (none) -> -; Vendor 1 (none) -> Digikey; Vendor 1 Part no. (none) -> 311-47.5KCRCT-ND; Vendor 2 (none) -> LCSC
- R210, R213, R214: footprint (none) -> Resistor_SMD:R_0805_2012Metric_Pad1.20x1.40mm_HandSolder; Manufacturer (none) -> -; Manufacturer Part no. (none) -> -; Vendor 1 (none) -> Digikey; Vendor 1 Part no. (none) -> 311-1.00KCRCT-ND; Vendor 2 (none) -> LCSC
- R211, R212: footprint (none) -> Resistor_SMD:R_0805_2012Metric_Pad1.20x1.40mm_HandSolder; Manufacturer (none) -> -; Manufacturer Part no. (none) -> -; Vendor 1 (none) -> Digikey; Vendor 1 Part no. (none) -> 311-10.0KCRCT-ND; Vendor 2 (none) -> LCSC

Commit message: Mod: Changed parts to match with both vendors
Parts:
- C201, C206, C207, C208: Manufacturer - -> Samsung Electro-Mechanics; Manufacturer Part no. - -> CL21B104KBCNFNC; Vendor 2 Part no. (none) -> C318718
- C202, C204, C205: Manufacturer - -> Samsung Electro-Mechanics; Manufacturer Part no. - -> CL21A106KOQNNNE; Vendor 2 Part no. (none) -> C1713
- C203: Manufacturer - -> Samsung Electro-Mechanics; Manufacturer Part no. - -> CL21B105KPFNNNE; Vendor 2 Part no. (none) -> C107367
- D201: footprint Package_TO_SOT_SMD:SOT-143 -> Package_TO_SOT_SMD:SOT-143_Handsoldering; Manufacturer - -> Littelfuse Inc.; Vendor 2 Part no. C7074 -> C7074
- D202, D203: Manufacturer - -> Lite-On Inc.; Manufacturer Part no. - -> LTST-C171GKT; Vendor 2 Part no. (none) -> C913075
- J201: Vendor 2 Part no. C3020560 -> C3020560
- Q201, Q202: Comment (none) -> General purpose NPN transistor
- R201, R204, R205, R208, R209: Manufacturer - -> YAGEO; Manufacturer Part no. - -> RC0805JR-070RL; Vendor 2 Part no. (none) -> C96345
- R202, R203: Manufacturer - -> YAGEO; Manufacturer Part no. - -> RC0805FR-075K1L; Vendor 2 Part no. (none) -> C84375
- R206: Manufacturer - -> YAGEO; Manufacturer Part no. - -> RC0805FR-0722K1L; Vendor 2 Part no. (none) -> C273840
- R207: Manufacturer - -> YAGEO; Manufacturer Part no. - -> RC0805FR-0747K5L; Vendor 2 Part no. (none) -> C137519
- R210, R213, R214: Manufacturer - -> YAGEO; Manufacturer Part no. - -> RC0805FR-071KL; Vendor 2 Part no. (none) -> C95781
- R211, R212: Manufacturer - -> YAGEO; Manufacturer Part no. - -> RC0805FR-0710KL; Vendor 2 Part no. (none) -> C84376
- U201: footprint Package_DFN_QFN:QFN-24-1EP_4x4mm_P0.5mm_EP2.6x2.6mm -> Package_DFN_QFN:QFN-24-1EP_4x4mm_P0.5mm_EP2.6x2.6mm_ThermalVias; Vendor 2 Part no. C969151 -> C969151
