File: src/USB.kicad_sch (KiCad schematic)
At the start: 29 parts, among them J201 USB_C_Receptacle_USB2.0_16P, Q201 NPN BJT, Q202 NPN BJT, U201 CP2102N-Axx-xQFN24

Commit message: Add: JLCPCB Database and selected components for the assembly
Parts:
- C201, C206, C207, C208: Comment (none) -> Best fit from the JLCPCB "Basic" compontens; Manufacturer Part no. CL21B104KBCNFNC -> CL21B104KCFNNNE; Vendor 1 Part no. 1276-2444-1-ND -> 1276-6840-1-ND; Vendor 2 Part no. C318718 -> C28233
- C202, C203, C204, C205, R201, R202, R203, R204, R205, R208, R209, R210, R211, R212, R213, R214: Comment (none) -> Best fit from the JLCPCB "Basic" compontens
- D201: LCSC (none) -> C7074
- D202, D203: LCSC (none) -> C913075
- J201: LCSC (none) -> C3020560
- Q201, Q202: LCSC (none) -> C49581
- R206: LCSC (none) -> C17552
- R207: LCSC (none) -> C26011
- U201: LCSC (none) -> C969151

Commit message: Fix: Part no. of D201, because it was the wrong one
Parts:
- D201: value SP0503BAHT -> SP0503BAHTG
Changed lines of the file:
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@@
 	(title_block
 		(title "Wordclock - USB & UART")
-		(date "2024-11-17")
+		(date "2024-11-25")
 		(rev "A")
 		(company "ElektroNik Zoller")
@@
 			)
 		)
-		(property "Value" "SP0503BAHT"
+		(property "Value" "SP0503BAHTG"
 			(at 69.85 107.9499 0)
 			(effects
@@
 			(effects
 				(font
+					(size 1.27 1.27)
+				)
+				(hide yes)
+			)
+		)
+		(property "Internal 1 Part no." ""
+			(at 76.2 106.68 0)
+			(effects
+				(font
+					(size 1.27 1.27)
+				)
+				(hide yes)
+			)
+		)
+		(property "Internal 2 Part no." ""
+			(at 76.2 106.68 0)
+			(effects
+				(font
+					(size 1.27 1.27)
+				)
+				(hide yes)
+			)
+		)
+		(property "Comment" ""
+			(at 76.2 106.68 0)
+			(effects
+				(font

Commit message: Mod: Updated date and fixed some typo
Parts:
- C201, C202, C203, C204, C205, C206, C207, C208, R201, R202, R203, R204, R205, R208, R209, R210, R211, R212, R213, R214: Comment Best fit from the JLCPCB "Basic" compontens -> Best fit from the JLCPCB "Basic" components
Changed lines of the file:
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@@
 			)
 		)
-		(property "Comment" "Best fit from the JLCPCB \"Basic\" compontens"
+		(property "Comment" "Best fit from the JLCPCB \"Basic\" components"
 			(at 190.5 71.12 0)
 			(effects
@@
 			)
 		)
-		(property "Comment" "Best fit from the JLCPCB \"Basic\" compontens"
+		(property "Comment" "Best fit from the JLCPCB \"Basic\" components"
 			(at 139.7 177.8 0)
 			(effects
@@
 			)
 		)
-		(property "Comment" "Best fit from the JLCPCB \"Basic\" compontens"
+		(property "Comment" "Best fit from the JLCPCB \"Basic\" components"
 			(at 69.85 71.12 0)
 			(effects
@@
 			)
 		)
-		(property "Comment" "Best fit from the JLCPCB \"Basic\" compontens"
+		(property "Comment" "Best fit from the JLCPCB \"Basic\" components"
 			(at 152.4 177.8 0)
 			(effects
@@
 			)
 		)
-		(property "Comment" "Best fit from the JLCPCB \"Basic\" compontens "
+		(property "Comment" "Best fit from the JLCPCB \"Basic\" components "
 			(at 31.75 113.03 0)
 			(effects
@@
 			)
 		)
-		(property "Comment" "Best fit from the JLCPCB \"Basic\" compontens"
+		(property "Comment" "Best fit from the JLCPCB \"Basic\" components"
 			(at 25.4 113.03 0)
 			(effects
@@
 			)
 		)
-		(property "Comment" "Best fit from the JLCPCB \"Basic\" compontens"
+		(property "Comment" "Best fit from the JLCPCB \"Basic\" components"
 			(at 266.7 80.01 0)
 			(effects
@@
 			)
 		)
-		(property "Comment" "Best fit from the JLCPCB \"Basic\" compontens "
+		(property "Comment" "Best fit from the JLCPCB \"Basic\" components "
 			(at 114.3 83.82 0)
 			(effects
@@
 			)
 		)
-		(property "Comment" "Best fit from the JLCPCB \"Basic\" compontens"
+		(property "Comment" "Best fit from the JLCPCB \"Basic\" components"
 			(at 165.1 177.8 0)
 			(effects
@@
 			)
 		)
-		(property "Comment" "Best fit from the JLCPCB \"Basic\" compontens "
+		(property "Comment" "Best fit from the JLCPCB \"Basic\" components "
 			(at 93.98 101.6 0)
 			(effects
@@
 			)
 		)
-		(property "Comment" "Best fit from the JLCPCB \"Basic\" compontens"
+		(property "Comment" "Best fit from the JLCPCB \"Basic\" components"
 			(at 114.3 63.5 0)
 			(effects
@@
 			)
 		)
-		(property "Comment" "Best fit from the JLCPCB \"Basic\" compontens "
+		(property "Comment" "Best fit from the JLCPCB \"Basic\" components "
 			(at 114.3 177.8 0)
 			(effects
@@
 			)
 		)
-		(property "Comment" "Best fit from the JLCPCB \"Basic\" compontens"
+		(property "Comment" "Best fit from the JLCPCB \"Basic\" components"
 			(at 69.85 73.66 0)
 			(effects
@@
 			)
 		)
-		(property "Comment" "Best fit from the JLCPCB \"Basic\" compontens "
+		(property "Comment" "Best fit from the JLCPCB \"Basic\" components "
 			(at 96.52 101.6 0)
 			(effects
@@
 			)
 		)
-		(property "Comment" "Best fit from the JLCPCB \"Basic\" compontens "
+		(property "Comment" "Best fit from the JLCPCB \"Basic\" components "
 			(at 101.6 177.8 0)
 			(effects
@@
 			)
 		)
-		(property "Comment" "Best fit from the JLCPCB \"Basic\" compontens"
+		(property "Comment" "Best fit from the JLCPCB \"Basic\" components"
 			(at 254 80.01 0)
 			(effects
@@
 			)
 		)
-		(property "Comment" "Best fit from the JLCPCB \"Basic\" compontens"
+		(property "Comment" "Best fit from the JLCPCB \"Basic\" components"
 			(at 133.35 59.69 0)
 			(effects
@@
 			)
 		)
-		(property "Comment" "Best fit from the JLCPCB \"Basic\" compontens "
+		(property "Comment" "Best fit from the JLCPCB \"Basic\" components "
 			(at 127 177.8 0)
 			(effects
@@
 			)
 		)
-		(property "Comment" "Best fit from the JLCPCB \"Basic\" compontens "
+		(property "Comment" "Best fit from the JLCPCB \"Basic\" components "
 			(at 114.3 81.28 0)
 			(effects
@@
 			)
 		)
-		(property "Comment" "Best fit from the JLCPCB \"Basic\" compontens"
+		(property "Comment" "Best fit from the JLCPCB \"Basic\" components"
 			(at 190.5 87.63 0)
 			(effects
