File: src/RTC.kicad_sch (KiCad schematic)
At the start: 11 parts, among them U401 DS3231M

Commit message: Add: JLCPCB Database and selected components for the assembly
Parts:
- BT401: LCSC (none) -> C6379018
- C401, C403, R401, R402, R403, R404, R405: Comment (none) -> Best fit from the JLCPCB "Basic" compontens
- C402, C404: Comment (none) -> Best fit from the JLCPCB "Basic" compontens; Manufacturer Part no. CL21B104KBCNFNC -> CL21B104KCFNNNE; Vendor 1 Part no. 1276-2444-1-ND -> 1276-6840-1-ND; Vendor 2 Part no. C318718 -> C28233
- U401: LCSC (none) -> C107410
Changed lines of the file:
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@@
 	(title_block
 		(title "Wordclock - Real Time Clock")
-		(date "2024-11-01")
+		(date "2024-11-17")
 		(rev "A")
 		(company "ElektroNik Zoller")
@@
 			)
 		)
-		(property "Manufacturer Part no." "CL21B104KBCNFNC"
+		(property "Manufacturer Part no." "CL21B104KCFNNNE"
 			(at 165.1 177.8 0)
 			(effects
@@
 			)
 		)
-		(property "Vendor 1 Part no." "1276-2444-1-ND "
+		(property "Vendor 1 Part no." "1276-6840-1-ND"
 			(at 165.1 177.8 0)
 			(effects
@@
 			)
 		)
-		(property "Vendor 2 Part no." "C318718"
+		(property "Vendor 2 Part no." "C28233"
 			(at 165.1 177.8 0)
 			(effects
@@
 			)
 		)
+		(property "Comment" "Best fit from the JLCPCB \"Basic\" compontens"
+			(at 165.1 177.8 0)
+			(effects
+				(font
+					(size 1.27 1.27)
+				)
+				(hide yes)
+			)
+		)
 		(pin "2"
 		)
@@
 			)
 		)
+		(property "LCSC" "C6379018"
+			(at 0 175.26 0)
+			(effects
+				(font
+					(size 1.27 1.27)
+				)
+				(hide yes)
+			)
+		)
 		(pin "2"
 		)
@@
 			)
 		)
+		(property "Comment" "Best fit from the JLCPCB \"Basic\" compontens"
+			(at 146.05 74.93 0)
+			(effects
+				(font
+					(size 1.27 1.27)
+				)
+				(hide yes)
+			)
+		)
 		(pin "1"
 		)
@@
 			)
 		)
+		(property "Comment" "Best fit from the JLCPCB \"Basic\" compontens "
+			(at 165.1 81.28 0)
+			(effects
+				(font
+					(size 1.27 1.27)
+				)
+				(hide yes)
+			)
+		)
 		(pin "2"
 		)
@@
 			)
 		)
+		(property "Comment" "Best fit from the JLCPCB \"Basic\" compontens "
+			(at 165.1 88.9 0)
+			(effects
+				(font
+					(size 1.27 1.27)
+				)
+				(hide yes)
+			)
+		)
 		(pin "2"
 		)
@@
 			)
 		)
+		(property "Comment" "Best fit from the JLCPCB \"Basic\" compontens "
+			(at 25.4 177.8 0)
+			(effects
+				(font
+					(size 1.27 1.27)
+				)
+				(hide yes)
+			)
+		)
 		(pin "2"
 		)
@@
 			)
 		)
+		(property "Comment" "Best fit from the JLCPCB \"Basic\" compontens"
+			(at 133.35 74.93 0)
+			(effects
+				(font
+					(size 1.27 1.27)
+				)
+				(hide yes)
+			)
+		)
 		(pin "1"
 		)
@@
 			)
 		)
+		(property "Comment" "Best fit from the JLCPCB \"Basic\" compontens "
+			(at 88.9 91.44 0)
+			(effects
+				(font
+					(size 1.27 1.27)
+				)
+				(hide yes)
+			)
+		)
 		(pin "2"
 		)
@@
 			)
 		)
+		(property "LCSC" "C107410"
+			(at 0 172.72 0)
+			(effects
+				(font
+					(size 1.27 1.27)
+				)
+				(hide yes)
+			)
+		)
 		(pin "12"
 		)
@@
 			)
 		)
+		(property "Comment" "Best fit from the JLCPCB \"Basic\" compontens"
+			(at 152.4 177.8 0)
+			(effects
+				(font
+					(size 1.27 1.27)
+				)
+				(hide yes)
+			)
+		)
 		(pin "2"
 		)
@@
 			)
 		)
-		(property "Manufacturer Part no." "CL21B104KBCNFNC"
+		(property "Manufacturer Part no." "CL21B104KCFNNNE"
 			(at 38.1 177.8 0)
 			(effects
@@
 			)
 		)
-		(property "Vendor 1 Part no." "1276-2444-1-ND "
+		(property "Vendor 1 Part no." "1276-6840-1-ND"
 			(at 38.1 177.8 0)
 			(effects
@@
 			)
 		)
-		(property "Vendor 2 Part no." "C318718"
+		(property "Vendor 2 Part no." "C28233"
+			(at 38.1 177.8 0)
+			(effects
+				(font
+					(size 1.27 1.27)
+				)
+				(hide yes)
+			)
+		)
+		(property "Comment" "Best fit from the JLCPCB \"Basic\" compontens"
 			(at 38.1 177.8 0)
 			(effects

Commit message: Fix: JLCPCB production data to be correct for production
Parts:
- U401: Comment LCSC, only has the 8 pin variant -> LCSC, only has the compatible DS3231SN in stock; Vendor 2 Part no. C107410 -> C9866
Changed lines of the file:
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@@
 			)
 		)
-		(property "Vendor 2 Part no." "C107410"
+		(property "Vendor 2 Part no." "C9866"
 			(at 114.3 86.36 0)
 			(effects
@@
 			)
 		)
-		(property "Comment" "LCSC, only has the 8 pin variant"
+		(property "Comment" "LCSC, only has the compatible DS3231SN in stock"
 			(at 114.3 86.36 0)
 			(effects
