File: src/RTC.kicad_sch (KiCad schematic)
At the start: 11 parts, among them U401 DS3231M

Commit message: Mod: Updated date and fixed some typo
Parts:
- C401, C402, C403, C404, R401, R402, R403, R404, R405: Comment Best fit from the JLCPCB "Basic" compontens -> Best fit from the JLCPCB "Basic" components
Changed lines of the file:
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@@
 	(title_block
 		(title "Wordclock - Real Time Clock")
-		(date "2024-11-17")
+		(date "2024-11-25")
 		(rev "A")
 		(company "ElektroNik Zoller")
@@
 			)
 		)
-		(property "Comment" "Best fit from the JLCPCB \"Basic\" compontens"
+		(property "Comment" "Best fit from the JLCPCB \"Basic\" components"
 			(at 165.1 177.8 0)
 			(effects
@@
 			)
 		)
-		(property "Comment" "Best fit from the JLCPCB \"Basic\" compontens"
+		(property "Comment" "Best fit from the JLCPCB \"Basic\" components"
 			(at 146.05 74.93 0)
 			(effects
@@
 			)
 		)
-		(property "Comment" "Best fit from the JLCPCB \"Basic\" compontens "
+		(property "Comment" "Best fit from the JLCPCB \"Basic\" components "
 			(at 165.1 81.28 0)
 			(effects
@@
 			)
 		)
-		(property "Comment" "Best fit from the JLCPCB \"Basic\" compontens "
+		(property "Comment" "Best fit from the JLCPCB \"Basic\" components "
 			(at 165.1 88.9 0)
 			(effects
@@
 			)
 		)
-		(property "Comment" "Best fit from the JLCPCB \"Basic\" compontens "
+		(property "Comment" "Best fit from the JLCPCB \"Basic\" components "
 			(at 25.4 177.8 0)
 			(effects
@@
 			)
 		)
-		(property "Comment" "Best fit from the JLCPCB \"Basic\" compontens"
+		(property "Comment" "Best fit from the JLCPCB \"Basic\" components"
 			(at 133.35 74.93 0)
 			(effects
@@
 			)
 		)
-		(property "Comment" "Best fit from the JLCPCB \"Basic\" compontens "
+		(property "Comment" "Best fit from the JLCPCB \"Basic\" components "
 			(at 88.9 91.44 0)
 			(effects
@@
 			)
 		)
-		(property "Comment" "Best fit from the JLCPCB \"Basic\" compontens"
+		(property "Comment" "Best fit from the JLCPCB \"Basic\" components"
 			(at 152.4 177.8 0)
 			(effects
@@
 			)
 		)
-		(property "Comment" "Best fit from the JLCPCB \"Basic\" compontens"
+		(property "Comment" "Best fit from the JLCPCB \"Basic\" components"
 			(at 38.1 177.8 0)
 			(effects
