File: src/BrightnessSensor.kicad_sch (KiCad schematic)
At the start: 12 parts, among them U501 BH1750xxx-xx

Commit message: Mod: Checked a few things and added the power limitation text to the LEDs page
Parts:
- renumbered C504 to C501, C505 to C502, C501 to C503, C502 to C504, C503 to C505, R505 to R501, R504 to R502, R501 to R503, R503 to R504, R502 to R505

Commit message: Add: Vendor no. and footprints
Parts:
- C501, C503: footprint (none) -> Capacitor_SMD:C_0805_2012Metric_Pad1.18x1.45mm_HandSolder; Manufacturer (none) -> -; Manufacturer Part no. (none) -> -; Vendor 1 (none) -> Digikey; Vendor 1 Part no. (none) -> 1276-1096-1-ND; Vendor 2 (none) -> LCSC
- C502, C504: footprint (none) -> Capacitor_SMD:C_0805_2012Metric_Pad1.18x1.45mm_HandSolder; Manufacturer (none) -> -; Manufacturer Part no. (none) -> -; Vendor 1 (none) -> Digikey; Vendor 1 Part no. (none) -> 1276-2444-1-ND; Vendor 2 (none) -> LCSC
- C505: footprint (none) -> Capacitor_SMD:C_0805_2012Metric_Pad1.18x1.45mm_HandSolder; Manufacturer (none) -> -; Manufacturer Part no. (none) -> -; Vendor 1 (none) -> Digikey; Vendor 1 Part no. (none) -> 1276-1275-2-ND; Vendor 2 (none) -> LCSC
- JP501, R502: Manufacturer (none) -> -; Manufacturer Part no. (none) -> -; Vendor 1 (none) -> -; Vendor 1 Part no. (none) -> -; Vendor 2 (none) -> -; Vendor 2 Part no. (none) -> -
- R501, R505: footprint (none) -> Resistor_SMD:R_0805_2012Metric_Pad1.20x1.40mm_HandSolder; Manufacturer (none) -> -; Manufacturer Part no. (none) -> -; Vendor 1 (none) -> Digikey; Vendor 1 Part no. (none) -> 311-10.0KCRCT-ND; Vendor 2 (none) -> LCSC
- R503: footprint (none) -> Resistor_SMD:R_0805_2012Metric_Pad1.20x1.40mm_HandSolder; Manufacturer (none) -> -; Manufacturer Part no. (none) -> -; Vendor 1 (none) -> Digikey; Vendor 1 Part no. (none) -> 311-0.0ARCT-ND; Vendor 2 (none) -> LCSC
- R504: footprint (none) -> Resistor_SMD:R_0805_2012Metric_Pad1.20x1.40mm_HandSolder; Manufacturer (none) -> -; Manufacturer Part no. (none) -> -; Vendor 1 (none) -> Digikey; Vendor 1 Part no. (none) -> 311-1.00KCRCT-ND; Vendor 2 (none) -> LCSC
- U501: Manufacturer (none) -> Rohm Semiconductor; Manufacturer Part no. (none) -> BH1750FVI-TR; Vendor 1 (none) -> Digikey; Vendor 1 Part no. (none) -> BH1750FVICT-ND; Vendor 2 (none) -> LCSC; Vendor 2 Part no. (none) -> C78960

Commit message: Mod: Changed parts to match with both vendors
Parts:
- C501, C503: Manufacturer - -> Samsung Electro-Mechanics; Manufacturer Part no. - -> CL21A106KOQNNNE; Vendor 2 Part no. (none) -> C1713
- C502, C504: Manufacturer - -> Samsung Electro-Mechanics; Manufacturer Part no. - -> CL21B104KBCNFNC; Vendor 2 Part no. (none) -> C318718
- C505: Manufacturer - -> Samsung Electro-Mechanics; Manufacturer Part no. - -> CL21B105KPFNNNE; Vendor 2 Part no. (none) -> C107367
- R501, R505: Manufacturer - -> YAGEO; Manufacturer Part no. - -> RC0805FR-0710KL; Vendor 2 Part no. (none) -> C84376
- R503: Manufacturer - -> YAGEO; Manufacturer Part no. - -> RC0805JR-070RL; Vendor 2 Part no. (none) -> C96345
- R504: Manufacturer - -> YAGEO; Manufacturer Part no. - -> RC0805FR-071KL; Vendor 2 Part no. (none) -> C95781
Changed lines of the file:
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@@
 	(title_block
 		(title "Wordclock - Brightness Sensor")
-		(date "2024-10-27")
+		(date "2024-10-29")
 		(rev "A")
 		(company "ElektroNik Zoller")
@@
 			)
 		)
-		(property "Manufacturer" "-"
+		(property "Manufacturer" "YAGEO"
 			(at 88.9 82.55 0)
 			(effects
@@
 			)
 		)
-		(property "Manufacturer Part no." "-"
+		(property "Manufacturer Part no." "RC0805FR-0710KL"
 			(at 88.9 82.55 0)
 			(effects
@@
 			)
 		)
-		(property "Vendor 2 Part no." ""
+		(property "Vendor 2 Part no." "C84376"
 			(at 88.9 82.55 0)
 			(effects
@@
 			)
 		)
-		(property "Manufacturer" "-"
+		(property "Manufacturer" "Samsung Electro-Mechanics"
 			(at 184.15 99.06 0)
 			(effects
@@
 			)
 		)
-		(property "Manufacturer Part no." "-"
+		(property "Manufacturer Part no." "CL21B105KPFNNNE"
 			(at 184.15 99.06 0)
 			(effects
@@
 			)
 		)
+		(property "Vendor 2 Part no." "C107367"
+			(at 184.15 99.06 0)
+			(effects
+				(font
+					(size 1.27 1.27)
+				)
+				(hide yes)
+			)
+		)
 		(pin "2"
 		)
@@
 			)
 		)
-		(property "Manufacturer" "-"
+		(property "Manufacturer" "Samsung Electro-Mechanics"
 			(at 165.1 177.8 0)
 			(effects
@@
 			)
 		)
-		(property "Manufacturer Part no." "-"
+		(property "Manufacturer Part no." "CL21B104KBCNFNC"
 			(at 165.1 177.8 0)
 			(effects
@@
 			)
 		)
+		(property "Vendor 2 Part no." "C318718"
+			(at 165.1 177.8 0)
+			(effects
+				(font
+					(size 1.27 1.27)
+				)
+				(hide yes)
+			)
+		)
 		(pin "2"
 		)
@@
 			)
 		)
-		(property "Manufacturer" "-"
+		(property "Manufacturer" "YAGEO"
 			(at 171.45 88.9 0)
 			(effects
@@
 			)
 		)
-		(property "Manufacturer Part no." "-"
+		(property "Manufacturer Part no." "RC0805JR-070RL"
 			(at 171.45 88.9 0)
 			(effects
@@
 			)
 		)
-		(property "Vendor 2 Part no." ""
+		(property "Vendor 2 Part no." "C96345"
 			(at 171.45 88.9 0)
 			(effects
@@
 			)
 		)
-		(property "Manufacturer" "-"
+		(property "Manufacturer" "YAGEO"
 			(at 184.15 81.28 0)
 			(effects
@@
 			)
 		)
-		(property "Manufacturer Part no." "-"
+		(property "Manufacturer Part no." "RC0805FR-071KL"
 			(at 184.15 81.28 0)
 			(effects
@@
 			)
 		)
+		(property "Vendor 2 Part no." "C95781"
+			(at 184.15 81.28 0)
+			(effects
+				(font
+					(size 1.27 1.27)
+				)
+				(hide yes)
+			)
+		)
 		(pin "1"
 		)
@@
 			)
 		)
-		(property "Manufacturer" "-"
+		(property "Manufacturer" "Samsung Electro-Mechanics"
 			(at 38.1 177.8 0)
 			(effects
@@
 			)
 		)
-		(property "Manufacturer Part no." "-"
+		(property "Manufacturer Part no." "CL21B104KBCNFNC"
 			(at 38.1 177.8 0)
 			(effects
@@
 			)
 		)
-		(property "Vendor 2 Part no." ""
+		(property "Vendor 2 Part no." "C318718"
 			(at 38.1 177.8 0)
 			(effects
@@
 			)
 		)
-		(property "Manufacturer" "-"
+		(property "Manufacturer" "Samsung Electro-Mechanics"
 			(at 152.4 177.8 0)
 			(effects
@@
 			)
 		)
-		(property "Manufacturer Part no." "-"
+		(property "Manufacturer Part no." "CL21A106KOQNNNE"
 			(at 152.4 177.8 0)
 			(effects
@@
 			)
 		)
+		(property "Vendor 2 Part no." "C1713"
+			(at 152.4 177.8 0)
+			(effects
+				(font
+					(size 1.27 1.27)
+				)
+				(hide yes)
+			)
+		)
 		(pin "2"
 		)
@@
 			)
 		)
-		(property "Manufacturer" "-"
+		(property "Manufacturer" "Samsung Electro-Mechanics"
 			(at 25.4 177.8 0)
 			(effects
@@
 			)
 		)
-		(property "Manufacturer Part no." "-"
+		(property "Manufacturer Part no." "CL21A106KOQNNNE"
 			(at 25.4 177.8 0)
 			(effects
@@
 			)
 		)
-		(property "Vendor 2 Part no." ""
+		(property "Vendor 2 Part no." "C1713"
 			(at 25.4 177.8 0)
 			(effects
@@
 			)
 		)
-		(property "Manufacturer" "-"
+		(property "Manufacturer" "YAGEO"
 			(at 196.85 99.06 0)
 			(effects
@@
 			)
 		)
-		(property "Manufacturer Part no." "-"
+		(property "Manufacturer Part no." "RC0805FR-0710KL"
 			(at 196.85 99.06 0)
 			(effects
@@
 			(at 196.85 99.06 0)
 			(effects
+				(font
+					(size 1.27 1.27)
+				)
+				(hide yes)
+			)
+		)
+		(property "Vendor 2 Part no." "C84376"
+			(at 196.85 99.06 0)
+			(effects

Commit message: Add: JLCPCB Database and selected components for the assembly
Parts:
- C501, C503, C505, R501, R503, R504, R505: Comment (none) -> Best fit from the JLCPCB "Basic" compontens
- C502, C504: Comment (none) -> Best fit from the JLCPCB "Basic" compontens; Manufacturer Part no. CL21B104KBCNFNC -> CL21B104KCFNNNE; Vendor 1 Part no. 1276-2444-1-ND -> 1276-6840-1-ND; Vendor 2 Part no. C318718 -> C28233
- U501: LCSC (none) -> C78960
Changed lines of the file:
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@@
 	(title_block
 		(title "Wordclock - Brightness Sensor")
-		(date "2024-10-29")
+		(date "2024-11-17")
 		(rev "A")
 		(company "ElektroNik Zoller")
@@
 			)
 		)
+		(property "Comment" "Best fit from the JLCPCB \"Basic\" compontens"
+			(at 88.9 82.55 0)
+			(effects
+				(font
+					(size 1.27 1.27)
+				)
+				(hide yes)
+			)
+		)
 		(pin "1"
 		)
@@
 			)
 		)
+		(property "Comment" "Best fit from the JLCPCB \"Basic\" compontens"
+			(at 184.15 99.06 0)
+			(effects
+				(font
+					(size 1.27 1.27)
+				)
+				(hide yes)
+			)
+		)
 		(pin "2"
 		)
@@
 			)
 		)
-		(property "Manufacturer Part no." "CL21B104KBCNFNC"
+		(property "Manufacturer Part no." "CL21B104KCFNNNE"
 			(at 165.1 177.8 0)
 			(effects
@@
 			)
 		)
-		(property "Vendor 1 Part no." "1276-2444-1-ND "
+		(property "Vendor 1 Part no." "1276-6840-1-ND"
 			(at 165.1 177.8 0)
 			(effects
@@
 			)
 		)
-		(property "Vendor 2 Part no." "C318718"
+		(property "Vendor 2 Part no." "C28233"
+			(at 165.1 177.8 0)
+			(effects
+				(font
+					(size 1.27 1.27)
+				)
+				(hide yes)
+			)
+		)
+		(property "Comment" "Best fit from the JLCPCB \"Basic\" compontens"
 			(at 165.1 177.8 0)
 			(effects
@@
 			)
 		)
+		(property "LCSC" "C78960"
+			(at 457.2 172.72 0)
+			(effects
+				(font
+					(size 1.27 1.27)
+				)
+				(hide yes)
+			)
+		)
 		(pin "4"
 		)
@@
 			)
 		)
+		(property "Comment" "Best fit from the JLCPCB \"Basic\" compontens "
+			(at 171.45 88.9 0)
+			(effects
+				(font
+					(size 1.27 1.27)
+				)
+				(hide yes)
+			)
+		)
 		(pin "2"
 		)
@@
 			)
 		)
+		(property "Comment" "Best fit from the JLCPCB \"Basic\" compontens"
+			(at 184.15 81.28 0)
+			(effects
+				(font
+					(size 1.27 1.27)
+				)
+				(hide yes)
+			)
+		)
 		(pin "1"
 		)
@@
 			)
 		)
-		(property "Manufacturer Part no." "CL21B104KBCNFNC"
+		(property "Manufacturer Part no." "CL21B104KCFNNNE"
 			(at 38.1 177.8 0)
 			(effects
@@
 			)
 		)
-		(property "Vendor 1 Part no." "1276-2444-1-ND "
+		(property "Vendor 1 Part no." "1276-6840-1-ND"
 			(at 38.1 177.8 0)
 			(effects
@@
 			)
 		)
-		(property "Vendor 2 Part no." "C318718"
+		(property "Vendor 2 Part no." "C28233"
 			(at 38.1 177.8 0)
 			(effects
@@
 			)
 		)
+		(property "Comment" "Best fit from the JLCPCB \"Basic\" compontens"
+			(at 38.1 177.8 0)
+			(effects
+				(font
+					(size 1.27 1.27)
+				)
+				(hide yes)
+			)
+		)
 		(pin "2"
 		)
@@
 			)
 		)
+		(property "Comment" "Best fit from the JLCPCB \"Basic\" compontens "
+			(at 152.4 177.8 0)
+			(effects
+				(font
+					(size 1.27 1.27)
+				)
+				(hide yes)
+			)
+		)
 		(pin "2"
 		)
@@
 			)
 		)
+		(property "Comment" "Best fit from the JLCPCB \"Basic\" compontens "
+			(at 25.4 177.8 0)
+			(effects
+				(font
+					(size 1.27 1.27)
+				)
+				(hide yes)
+			)
+		)
 		(pin "2"
 		)
@@
 			(at 196.85 99.06 0)
 			(effects
+				(font
+					(size 1.27 1.27)
+				)
+				(hide yes)
+			)
+		)
+		(property "Comment" "Best fit from the JLCPCB \"Basic\" compontens"
+			(at 196.85 99.06 0)
+			(effects

Commit message: Mod: Updated date and fixed some typo
Parts:
- C501, C502, C503, C504, C505, R501, R503, R504, R505: Comment Best fit from the JLCPCB "Basic" compontens -> Best fit from the JLCPCB "Basic" components
Changed lines of the file:
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@@
 	(title_block
 		(title "Wordclock - Brightness Sensor")
-		(date "2024-11-17")
+		(date "2024-11-25")
 		(rev "A")
 		(company "ElektroNik Zoller")
@@
 			)
 		)
-		(property "Comment" "Best fit from the JLCPCB \"Basic\" compontens"
+		(property "Comment" "Best fit from the JLCPCB \"Basic\" components"
 			(at 88.9 82.55 0)
 			(effects
@@
 			)
 		)
-		(property "Comment" "Best fit from the JLCPCB \"Basic\" compontens"
+		(property "Comment" "Best fit from the JLCPCB \"Basic\" components"
 			(at 184.15 99.06 0)
 			(effects
@@
 			)
 		)
-		(property "Comment" "Best fit from the JLCPCB \"Basic\" compontens"
+		(property "Comment" "Best fit from the JLCPCB \"Basic\" components"
 			(at 165.1 177.8 0)
 			(effects
@@
 			)
 		)
-		(property "Comment" "Best fit from the JLCPCB \"Basic\" compontens "
+		(property "Comment" "Best fit from the JLCPCB \"Basic\" components "
 			(at 171.45 88.9 0)
 			(effects
@@
 			)
 		)
-		(property "Comment" "Best fit from the JLCPCB \"Basic\" compontens"
+		(property "Comment" "Best fit from the JLCPCB \"Basic\" components"
 			(at 184.15 81.28 0)
 			(effects
@@
 			)
 		)
-		(property "Comment" "Best fit from the JLCPCB \"Basic\" compontens"
+		(property "Comment" "Best fit from the JLCPCB \"Basic\" components"
 			(at 38.1 177.8 0)
 			(effects
@@
 			)
 		)
-		(property "Comment" "Best fit from the JLCPCB \"Basic\" compontens "
+		(property "Comment" "Best fit from the JLCPCB \"Basic\" components "
 			(at 152.4 177.8 0)
 			(effects
@@
 			)
 		)
-		(property "Comment" "Best fit from the JLCPCB \"Basic\" compontens "
+		(property "Comment" "Best fit from the JLCPCB \"Basic\" components "
 			(at 25.4 177.8 0)
 			(effects
@@
 			)
 		)
-		(property "Comment" "Best fit from the JLCPCB \"Basic\" compontens"
+		(property "Comment" "Best fit from the JLCPCB \"Basic\" components"
 			(at 196.85 99.06 0)
 			(effects
