File: src/LEDs.kicad_sch (KiCad schematic)
At the start: 3 parts, among them Q601 BSS138

Commit message: Mod: Checked a few things and added the power limitation text to the LEDs page
Parts:
- renumbered R602 to R601, R603 to R602
Changed lines of the file:
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@@
 	(title_block
 		(title "Wordclock - LEDs")
-		(date "2024-10-20")
+		(date "2024-10-27")
 		(rev "A")
 		(company "ElektroNik Zoller")
@@
 			(width 0)
 			(type default)
+		)
+	)
+	(text_box "Caution!\nNever use all LEDs at full brightness. This means that in normal clock mode between 10 and 30 LEDs will be on at the same time. At peak times these can be run at 100 % brightness without any problem. However, if the LEDs are used with other modes that control all 114 LEDs, the brightness must not exceed 50 %!\n\nOther applications need to be checked by the user. The USB connectors support up to 5V @ 3A (when using the appropriate PD power supply). Calculate about 20 mA per LED and per colour, i.e. a white LED (all colours combined) will consume about 60 mA. All 114 LEDs would therefore require more than 6.8A, which the USB PD (in this configuration) cannot provide!"
+		(exclude_from_sim no)
+		(at 13.97 177.8 0)
+		(size 161.29 17.78)
+		(stroke
+			(width 0)
+			(type default)
+		)
+		(fill
+			(type none)
+		)
+		(effects
+			(font
+				(size 1.27 1.27)
+			)
+			(justify left top)
 		)
 	)
@@
 		(dnp no)
 		(fields_autoplaced yes)
-		(property "Reference" "#PWR0603"
+		(property "Reference" "#PWR0602"
 			(at 50.8 29.21 0)
 			(effects
@@
 			(project "ESP-Wordclock"
 				(path "/bfaac094-0365-40a4-8b7a-d4d62ace544e/c23f8616-5eaa-4df3-8ee0-2a2271a82cce"
-					(reference "#PWR0603")
+					(reference "#PWR0602")
 					(unit 1)
 				)
@@
 		(dnp no)
 		(fields_autoplaced yes)
-		(property "Reference" "#PWR0602"
+		(property "Reference" "#PWR0603"
 			(at 63.5 29.21 0)
 			(effects
@@
 			(project "ESP-Wordclock"
 				(path "/bfaac094-0365-40a4-8b7a-d4d62ace544e/c23f8616-5eaa-4df3-8ee0-2a2271a82cce"
-					(reference "#PWR0602")
+					(reference "#PWR0603")
 					(unit 1)
 				)
@@
 		(on_board yes)
 		(dnp no)
-		(property "Reference" "R603"
+		(property "Reference" "R602"
 			(at 60.96 30.4799 0)
 			(effects
@@
 			(project "ESP-Wordclock"
 				(path "/bfaac094-0365-40a4-8b7a-d4d62ace544e/c23f8616-5eaa-4df3-8ee0-2a2271a82cce"
-					(reference "R603")
+					(reference "R602")
 					(unit 1)
 				)
@@
 		(dnp no)
 		(fields_autoplaced yes)
-		(property "Reference" "R602"
+		(property "Reference" "R601"
 			(at 40.64 30.4799 0)
 			(effects
@@
 			(project "ESP-Wordclock"
 				(path "/bfaac094-0365-40a4-8b7a-d4d62ace544e/c23f8616-5eaa-4df3-8ee0-2a2271a82cce"
-					(reference "R602")
+					(reference "R601")
 					(unit 1)
 				)

Commit message: Add: Vendor no. and footprints
Parts:
- Q601: Manufacturer (none) -> -; Manufacturer Part no. (none) -> BSS138; Vendor 1 (none) -> Digikey; Vendor 1 Part no. (none) -> BSS138CT-ND; Vendor 2 (none) -> LCSC; Vendor 2 Part no. (none) -> C518792
- R601, R602: footprint (none) -> Resistor_SMD:R_0805_2012Metric_Pad1.20x1.40mm_HandSolder; Manufacturer (none) -> -; Manufacturer Part no. (none) -> -; Vendor 1 (none) -> Digikey; Vendor 1 Part no. (none) -> 311-10.0KCRCT-ND; Vendor 2 (none) -> LCSC
Changed lines of the file:
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@@
+			)
+		)
+		(property "Vendor 1" "Digikey"
+			(at 50.8 35.56 0)
+			(effects
+				(font
+					(size 1.27 1.27)
+				)
+				(hide yes)
+			)
+		)
+		(property "Vendor 2" "LCSC"
+			(at 50.8 35.56 0)
+			(effects
+				(font
+					(size 1.27 1.27)
+				)
+				(hide yes)
+			)
+		)
+		(property "Manufacturer" "-"
+			(at 50.8 35.56 0)
+			(effects
+				(font
+					(size 1.27 1.27)
+				)
+				(hide yes)
+			)
+		)
+		(property "Manufacturer Part no." "BSS138"
+			(at 50.8 35.56 0)
+			(effects
+				(font
+					(size 1.27 1.27)
+				)
+				(hide yes)
+			)
+		)
+		(property "Vendor 1 Part no." "BSS138CT-ND"
+			(at 50.8 35.56 0)
+			(effects
+				(font
+					(size 1.27 1.27)
+				)
+				(hide yes)
+			)
+		)
+		(property "Vendor 2 Part no." " C518792"
+			(at 50.8 35.56 0)
+			(effects
+				(font
+					(size 1.27 1.27)
+				)
+				(hide yes)
 			)
 		)
@@
 			)
 		)
-		(property "Footprint" ""
+		(property "Footprint" "Resistor_SMD:R_0805_2012Metric_Pad1.20x1.40mm_HandSolder"
 			(at 65.278 31.75 90)
 			(effects
@@
 		)
 		(property "Sim.Type" ""
+			(at 63.5 31.75 0)
+			(effects
+				(font
+					(size 1.27 1.27)
+				)
+				(hide yes)
+			)
+		)
+		(property "Vendor 1" "Digikey"
+			(at 63.5 31.75 0)
+			(effects
+				(font
+					(size 1.27 1.27)
+				)
+				(hide yes)
+			)
+		)
+		(property "Vendor 2" "LCSC"
+			(at 63.5 31.75 0)
+			(effects
+				(font
+					(size 1.27 1.27)
+				)
+				(hide yes)
+			)
+		)
+		(property "Manufacturer" "-"
+			(at 63.5 31.75 0)
+			(effects
+				(font
+					(size 1.27 1.27)
+				)
+				(hide yes)
+			)
+		)
+		(property "Manufacturer Part no." "-"
+			(at 63.5 31.75 0)
+			(effects
+				(font
+					(size 1.27 1.27)
+				)
+				(hide yes)
+			)
+		)
+		(property "Vendor 1 Part no." "311-10.0KCRCT-ND"
 			(at 63.5 31.75 0)
 			(effects
@@
 			)
 		)
-		(property "Footprint" ""
+		(property "Footprint" "Resistor_SMD:R_0805_2012Metric_Pad1.20x1.40mm_HandSolder"
 			(at 36.322 31.75 90)
 			(effects
@@
 			(at 38.1 31.75 0)
 			(effects
+				(font
+					(size 1.27 1.27)
+				)
+				(hide yes)
+			)
+		)
+		(property "Vendor 1" "Digikey"
+			(at 38.1 31.75 0)
+			(effects
+				(font
+					(size 1.27 1.27)
+				)
+				(hide yes)
+			)
+		)
+		(property "Vendor 2" "LCSC"
+			(at 38.1 31.75 0)
+			(effects
+				(font
+					(size 1.27 1.27)
+				)
+				(hide yes)
+			)
+		)
+		(property "Manufacturer" "-"
+			(at 38.1 31.75 0)
+			(effects
+				(font
+					(size 1.27 1.27)
+				)
+				(hide yes)
+			)
+		)
+		(property "Manufacturer Part no." "-"
+			(at 38.1 31.75 0)
+			(effects
+				(font
+					(size 1.27 1.27)
+				)
+				(hide yes)
+			)
+		)
+		(property "Vendor 1 Part no." "311-10.0KCRCT-ND"
+			(at 38.1 31.75 0)
+			(effects

Commit message: Mod: Changed parts to match with both vendors
Parts:
- Q601: footprint Package_TO_SOT_SMD:SOT-23 -> Package_TO_SOT_SMD:SOT-23_Handsoldering; Comment (none) -> General purpose N-channel MOSFET; Vendor 2 Part no. C518792 -> C518792
- R601, R602: Manufacturer - -> YAGEO; Manufacturer Part no. - -> RC0805FR-0710KL; Vendor 2 Part no. (none) -> C84376
Changed lines of the file:
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@@
 	(title_block
 		(title "Wordclock - LEDs")
-		(date "2024-10-27")
+		(date "2024-10-29")
 		(rev "A")
 		(company "ElektroNik Zoller")
@@
 			)
 		)
-		(property "Footprint" "Package_TO_SOT_SMD:SOT-23"
+		(property "Footprint" "Package_TO_SOT_SMD:SOT-23_Handsoldering"
 			(at 48.895 40.64 0)
 			(effects
@@
 			)
 		)
-		(property "Vendor 2 Part no." " C518792"
+		(property "Vendor 2 Part no." "C518792"
+			(at 50.8 35.56 0)
+			(effects
+				(font
+					(size 1.27 1.27)
+				)
+				(hide yes)
+			)
+		)
+		(property "Comment" "General purpose N-channel MOSFET"
 			(at 50.8 35.56 0)
 			(effects
@@
 			)
 		)
-		(property "Manufacturer" "-"
+		(property "Manufacturer" "YAGEO"
 			(at 63.5 31.75 0)
 			(effects
@@
 			)
 		)
-		(property "Manufacturer Part no." "-"
+		(property "Manufacturer Part no." "RC0805FR-0710KL"
 			(at 63.5 31.75 0)
 			(effects
@@
 		)
 		(property "Vendor 1 Part no." "311-10.0KCRCT-ND"
+			(at 63.5 31.75 0)
+			(effects
+				(font
+					(size 1.27 1.27)
+				)
+				(hide yes)
+			)
+		)
+		(property "Vendor 2 Part no." "C84376"
 			(at 63.5 31.75 0)
 			(effects
@@
 			)
 		)
-		(property "Manufacturer" "-"
+		(property "Manufacturer" "YAGEO"
 			(at 38.1 31.75 0)
 			(effects
@@
 			)
 		)
-		(property "Manufacturer Part no." "-"
+		(property "Manufacturer Part no." "RC0805FR-0710KL"
 			(at 38.1 31.75 0)
 			(effects
@@
 			(at 38.1 31.75 0)
 			(effects
+				(font
+					(size 1.27 1.27)
+				)
+				(hide yes)
+			)
+		)
+		(property "Vendor 2 Part no." "C84376"
+			(at 38.1 31.75 0)
+			(effects

Commit message: Add: JLCPCB Database and selected components for the assembly
Parts:
- Q601: LCSC (none) -> C518792
- R601, R602: Comment (none) -> Best fit from the JLCPCB "Basic" compontens
Changed lines of the file:
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@@
 	(title_block
 		(title "Wordclock - LEDs")
-		(date "2024-10-29")
+		(date "2024-11-17")
 		(rev "A")
 		(company "ElektroNik Zoller")
@@
 			)
 		)
+		(property "LCSC" "C518792"
+			(at 15.24 -15.24 0)
+			(effects
+				(font
+					(size 1.27 1.27)
+				)
+				(hide yes)
+			)
+		)
 		(pin "3"
 		)
@@
 			)
 		)
+		(property "Comment" "Best fit from the JLCPCB \"Basic\" compontens"
+			(at 63.5 31.75 0)
+			(effects
+				(font
+					(size 1.27 1.27)
+				)
+				(hide yes)
+			)
+		)
 		(pin "2"
 		)
@@
 			(at 38.1 31.75 0)
 			(effects
+				(font
+					(size 1.27 1.27)
+				)
+				(hide yes)
+			)
+		)
+		(property "Comment" "Best fit from the JLCPCB \"Basic\" compontens"
+			(at 38.1 31.75 0)
+			(effects

Commit message: Mod: Updated date and fixed some typo
Parts:
- R601, R602: Comment Best fit from the JLCPCB "Basic" compontens -> Best fit from the JLCPCB "Basic" components
Changed lines of the file:
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@@
 	(title_block
 		(title "Wordclock - LEDs")
-		(date "2024-11-17")
+		(date "2024-11-25")
 		(rev "A")
 		(company "ElektroNik Zoller")
@@
 			)
 		)
-		(property "Comment" "Best fit from the JLCPCB \"Basic\" compontens"
+		(property "Comment" "Best fit from the JLCPCB \"Basic\" components"
 			(at 63.5 31.75 0)
 			(effects
@@
 			)
 		)
-		(property "Comment" "Best fit from the JLCPCB \"Basic\" compontens"
+		(property "Comment" "Best fit from the JLCPCB \"Basic\" components"
 			(at 38.1 31.75 0)
 			(effects
