File: src/MCU.kicad_sch (KiCad schematic)
At the start: 19 parts, among them SW301 SW_Push, SW302 SW_Push, U301 ESP32-C3-WROOM-02, U302 TLV1117LV33

Commit message: Add: JLCPCB Database and selected components for the assembly
Parts:
- C301, C305, C306, C309, R301, R302, R303, R304: Comment (none) -> Best fit from the JLCPCB "Basic" compontens
- C302, C303, C304, C307, C308: Comment (none) -> Best fit from the JLCPCB "Basic" compontens; Manufacturer Part no. CL21B104KBCNFNC -> CL21B104KCFNNNE; Vendor 1 Part no. 1276-2444-1-ND -> 1276-6840-1-ND; Vendor 2 Part no. C318718 -> C28233
- D301: LCSC (none) -> C284871
- D302: LCSC (none) -> C284931
- SW301, SW302: LCSC (none) -> C221896
- U301: LCSC (none) -> C2934560
- U302: LCSC (none) -> C15578
Changed lines of the file:
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@@
 	(title_block
 		(title "Wordclock - Microcontroller Unit & Power Supply")
-		(date "2024-10-29")
+		(date "2024-11-17")
 		(rev "A")
 		(company "ElektroNik Zoller")
@@
 			)
 		)
+		(property "Comment" "Best fit from the JLCPCB \"Basic\" compontens "
+			(at 241.3 69.85 0)
+			(effects
+				(font
+					(size 1.27 1.27)
+				)
+				(hide yes)
+			)
+		)
 		(pin "2"
 		)
@@
 			)
 		)
+		(property "LCSC" "C221896"
+			(at 121.92 121.92 0)
+			(effects
+				(font
+					(size 1.27 1.27)
+				)
+				(hide yes)
+			)
+		)
 		(pin "2"
 		)
@@
 			)
 		)
-		(property "Manufacturer Part no." "CL21B104KBCNFNC"
+		(property "Manufacturer Part no." "CL21B104KCFNNNE"
 			(at 203.2 69.85 0)
 			(effects
@@
 			)
 		)
-		(property "Vendor 1 Part no." "1276-2444-1-ND "
+		(property "Vendor 1 Part no." "1276-6840-1-ND"
 			(at 203.2 69.85 0)
 			(effects
@@
 			)
 		)
-		(property "Vendor 2 Part no." "C318718"
+		(property "Vendor 2 Part no." "C28233"
+			(at 203.2 69.85 0)
+			(effects
+				(font
+					(size 1.27 1.27)
+				)
+				(hide yes)
+			)
+		)
+		(property "Comment" "Best fit from the JLCPCB \"Basic\" compontens"
 			(at 203.2 69.85 0)
 			(effects
@@
 			)
 		)
+		(property "Comment" "Best fit from the JLCPCB \"Basic\" compontens"
+			(at 50.8 102.87 0)
+			(effects
+				(font
+					(size 1.27 1.27)
+				)
+				(hide yes)
+			)
+		)
 		(pin "2"
 		)
@@
 			)
 		)
+		(property "LCSC" "C221896"
+			(at 170.18 170.18 0)
+			(effects
+				(font
+					(size 1.27 1.27)
+				)
+				(hide yes)
+			)
+		)
 		(pin "2"
 		)
@@
 			)
 		)
+		(property "LCSC" "C284871"
+			(at 336.55 336.55 0)
+			(effects
+				(font
+					(size 1.27 1.27)
+				)
+				(hide yes)
+			)
+		)
 		(pin "1"
 		)
@@
 			)
 		)
+		(property "LCSC" "C284931"
+			(at 361.95 361.95 0)
+			(effects
+				(font
+					(size 1.27 1.27)
+				)
+				(hide yes)
+			)
+		)
 		(pin "1"
 		)
@@
 			)
 		)
-		(property "Manufacturer Part no." "CL21B104KBCNFNC"
+		(property "Manufacturer Part no." "CL21B104KCFNNNE"
 			(at 63.5 71.12 0)
 			(effects
@@
 			)
 		)
-		(property "Vendor 1 Part no." "1276-2444-1-ND "
+		(property "Vendor 1 Part no." "1276-6840-1-ND"
 			(at 63.5 71.12 0)
 			(effects
@@
 			)
 		)
-		(property "Vendor 2 Part no." "C318718"
+		(property "Vendor 2 Part no." "C28233"
 			(at 63.5 71.12 0)
 			(effects
@@
 			)
 		)
+		(property "Comment" "Best fit from the JLCPCB \"Basic\" compontens"
+			(at 63.5 71.12 0)
+			(effects
+				(font
+					(size 1.27 1.27)
+				)
+				(hide yes)
+			)
+		)
 		(pin "2"
 		)
@@
 			)
 		)
+		(property "Comment" "Best fit from the JLCPCB \"Basic\" compontens"
+			(at 228.6 120.65 0)
+			(effects
+				(font
+					(size 1.27 1.27)
+				)
+				(hide yes)
+			)
+		)
 		(pin "2"
 		)
@@
 			)
 		)
-		(property "Manufacturer Part no." "CL21B104KBCNFNC"
+		(property "Manufacturer Part no." "CL21B104KCFNNNE"
 			(at 38.1 177.8 0)
 			(effects
@@
 			)
 		)
-		(property "Vendor 1 Part no." "1276-2444-1-ND "
+		(property "Vendor 1 Part no." "1276-6840-1-ND"
 			(at 38.1 177.8 0)
 			(effects
@@
 			)
 		)
-		(property "Vendor 2 Part no." "C318718"
+		(property "Vendor 2 Part no." "C28233"
+			(at 38.1 177.8 0)
+			(effects
+				(font
+					(size 1.27 1.27)
+				)
+				(hide yes)
+			)
+		)
+		(property "Comment" "Best fit from the JLCPCB \"Basic\" compontens"
 			(at 38.1 177.8 0)
 			(effects
@@
 			)
 		)
+		(property "Comment" "Best fit from the JLCPCB \"Basic\" compontens "
+			(at 25.4 177.8 0)
+			(effects
+				(font
+					(size 1.27 1.27)
+				)
+				(hide yes)
+			)
+		)
 		(pin "2"
 		)
@@
 			)
 		)
+		(property "Comment" "Best fit from the JLCPCB \"Basic\" compontens"
+			(at 50.8 57.15 0)
+			(effects
+				(font
+					(size 1.27 1.27)
+				)
+				(hide yes)
+			)
+		)
 		(pin "2"
 		)
@@
 			)
 		)
+		(property "Comment" "Best fit from the JLCPCB \"Basic\" compontens"
+			(at 203.2 120.65 0)
+			(effects
+				(font
+					(size 1.27 1.27)
+				)
+				(hide yes)
+			)
+		)
 		(pin "2"
 		)
@@
 			)
 		)
+		(property "Comment" "Best fit from the JLCPCB \"Basic\" compontens "
+			(at 190.5 69.85 0)
+			(effects
+				(font
+					(size 1.27 1.27)
+				)
+				(hide yes)
+			)
+		)
 		(pin "2"
 		)
@@
 			)
 		)
+		(property "LCSC" "C2934560"
+			(at 0 203.2 0)
+			(effects
+				(font
+					(size 1.27 1.27)
+				)
+				(hide yes)
+			)
+		)
 		(pin "10"
 		)
@@
 			)
 		)
-		(property "Manufacturer Part no." "CL21B104KBCNFNC"
+		(property "Manufacturer Part no." "CL21B104KCFNNNE"
 			(at 63.5 119.38 0)
 			(effects
@@
 			)
 		)
-		(property "Vendor 1 Part no." "1276-2444-1-ND "
+		(property "Vendor 1 Part no." "1276-6840-1-ND"
 			(at 63.5 119.38 0)
 			(effects
@@
 			)
 		)
-		(property "Vendor 2 Part no." "C318718"
+		(property "Vendor 2 Part no." "C28233"
 			(at 63.5 119.38 0)
 			(effects
@@
 			)
 		)
+		(property "Comment" "Best fit from the JLCPCB \"Basic\" compontens"
+			(at 63.5 119.38 0)
+			(effects
+				(font
+					(size 1.27 1.27)
+				)
+				(hide yes)
+			)
+		)
 		(pin "2"
 		)
@@
 			)
 		)
-		(property "Manufacturer Part no." "CL21B104KBCNFNC"
+		(property "Manufacturer Part no." "CL21B104KCFNNNE"
 			(at 228.6 69.85 0)
 			(effects
@@
 			)
 		)
-		(property "Vendor 1 Part no." "1276-2444-1-ND "
+		(property "Vendor 1 Part no." "1276-6840-1-ND"
 			(at 228.6 69.85 0)
 			(effects
@@
 			)
 		)
-		(property "Vendor 2 Part no." "C318718"
+		(property "Vendor 2 Part no." "C28233"
+			(at 228.6 69.85 0)
+			(effects
+				(font
+					(size 1.27 1.27)
+				)
+				(hide yes)
+			)
+		)
+		(property "Comment" "Best fit from the JLCPCB \"Basic\" compontens"
 			(at 228.6 69.85 0)
 			(effects
@@
 			)
 		)
+		(property "Comment" "Best fit from the JLCPCB \"Basic\" compontens"
+			(at 76.2 71.12 0)
+			(effects
+				(font
+					(size 1.27 1.27)
+				)
+				(hide yes)
+			)
+		)
 		(pin "2"
 		)
@@
 			(effects
 				(font
+					(size 1.27 1.27)
+				)
+				(hide yes)
+			)
+		)
+		(property "LCSC" "C15578"
+			(at 0 127 0)
+			(effects
+				(font

Commit message: Mod: Updated date and fixed some typo
Parts:
- C301, C302, C303, C304, C305, C306, C307, C308, C309, R301, R302, R303, R304: Comment Best fit from the JLCPCB "Basic" compontens -> Best fit from the JLCPCB "Basic" components
Changed lines of the file:
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@@
 	(title_block
 		(title "Wordclock - Microcontroller Unit & Power Supply")
-		(date "2024-11-17")
+		(date "2024-11-25")
 		(rev "A")
 		(company "ElektroNik Zoller")
@@
 			)
 		)
-		(property "Comment" "Best fit from the JLCPCB \"Basic\" compontens "
+		(property "Comment" "Best fit from the JLCPCB \"Basic\" components "
 			(at 241.3 69.85 0)
 			(effects
@@
 			)
 		)
-		(property "Comment" "Best fit from the JLCPCB \"Basic\" compontens"
+		(property "Comment" "Best fit from the JLCPCB \"Basic\" components"
 			(at 203.2 69.85 0)
 			(effects
@@
 			)
 		)
-		(property "Comment" "Best fit from the JLCPCB \"Basic\" compontens"
+		(property "Comment" "Best fit from the JLCPCB \"Basic\" components"
 			(at 50.8 102.87 0)
 			(effects
@@
 			)
 		)
-		(property "Comment" "Best fit from the JLCPCB \"Basic\" compontens"
+		(property "Comment" "Best fit from the JLCPCB \"Basic\" components"
 			(at 63.5 71.12 0)
 			(effects
@@
 			)
 		)
-		(property "Comment" "Best fit from the JLCPCB \"Basic\" compontens"
+		(property "Comment" "Best fit from the JLCPCB \"Basic\" components"
 			(at 228.6 120.65 0)
 			(effects
@@
 			)
 		)
-		(property "Comment" "Best fit from the JLCPCB \"Basic\" compontens"
+		(property "Comment" "Best fit from the JLCPCB \"Basic\" components"
 			(at 38.1 177.8 0)
 			(effects
@@
 			)
 		)
-		(property "Comment" "Best fit from the JLCPCB \"Basic\" compontens "
+		(property "Comment" "Best fit from the JLCPCB \"Basic\" components "
 			(at 25.4 177.8 0)
 			(effects
@@
 			)
 		)
-		(property "Comment" "Best fit from the JLCPCB \"Basic\" compontens"
+		(property "Comment" "Best fit from the JLCPCB \"Basic\" components"
 			(at 50.8 57.15 0)
 			(effects
@@
 			)
 		)
-		(property "Comment" "Best fit from the JLCPCB \"Basic\" compontens"
+		(property "Comment" "Best fit from the JLCPCB \"Basic\" components"
 			(at 203.2 120.65 0)
 			(effects
@@
 			)
 		)
-		(property "Comment" "Best fit from the JLCPCB \"Basic\" compontens "
+		(property "Comment" "Best fit from the JLCPCB \"Basic\" components "
 			(at 190.5 69.85 0)
 			(effects
@@
 			)
 		)
-		(property "Comment" "Best fit from the JLCPCB \"Basic\" compontens"
+		(property "Comment" "Best fit from the JLCPCB \"Basic\" components"
 			(at 63.5 119.38 0)
 			(effects
@@
 			)
 		)
-		(property "Comment" "Best fit from the JLCPCB \"Basic\" compontens"
+		(property "Comment" "Best fit from the JLCPCB \"Basic\" components"
 			(at 228.6 69.85 0)
 			(effects
@@
 			)
 		)
-		(property "Comment" "Best fit from the JLCPCB \"Basic\" compontens"
+		(property "Comment" "Best fit from the JLCPCB \"Basic\" components"
 			(at 76.2 71.12 0)
 			(effects
