File: src/ESP-Wordclock.kicad_pcb (KiCad board)
At the start: 2 copper layers, 235 x 235 mm, 308 parts, among them J101 Conn_01x08_Pin, J201 USB_C_Receptacle_USB2.0_16P, Q201 NPN BJT, Q202 NPN BJT, Q601 BSS138, SW301 SW_Push, SW302 SW_Push, U201 CP2102N-Axx-xQFN24, U301 ESP32-C3-WROOM-02, U302 TLV1117LV33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

Commit message: Mod: Updated the whole PCB, run DRC and re-exported all manufacturing files
Parts:
- D201: value SP0503BAHT -> SP0503BAHTG
